File: template.kicad_sch (KiCad schematic)
At the start: 0 parts

Commit message: feat: :bookmark: add sheet metadata
Other:
- company: (none) -> Lukas Runge Veranstaltungstechnik
- title: (none) -> template
Changed lines of the file:
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@@
 	(generator_version "9.0")
 	(paper "A4")
+	(title_block
+		(title "template")
+		(rev "v0.0.1")
+		(company "Lukas Runge Veranstaltungstechnik")
+	)
 	(sheet_instances
 		(path "/"
